File: ESP_WeatherStation v2.0.sch (KiCad schematic (older format))
At the start: 21 parts, among them J1 Con1, J2 Conn_01x04, J3 Conn_01x04, U1 AZ1117-3.3, U2 ESP-12F, U3 Si7021, U4 BMP280

Commit message: Released version (PCB made)
Parts:
- U1: symbol ESP_WeatherStation-rescue:AZ1117-3.3 -> Regulator_Linear:AZ1117-3.3
- U2: symbol ESP_WeatherStation-rescue:ESP-12F -> ESP8266:ESP-12F
- U4: symbol ESP_WeatherStation-rescue:BMP280 -> ESP_WeatherStation-v2.0-rescue:MaxNil_components_BMP280-ESP_WeatherStation_v2.0-cache
Changed lines of the file:
@@
 EESchema Schematic File Version 4
+LIBS:ESP_WeatherStation v2.0-cache
 EELAYER 26 0
 EELAYER END
@@
 $EndComp
 $Comp
-L ESP_WeatherStation-rescue:AZ1117-3.3 U1
+L Regulator_Linear:AZ1117-3.3 U1
 U 1 1 5A92E9F5
 P 1700 1300
@@
 $EndComp
 $Comp
-L ESP_WeatherStation-rescue:BMP280 U4
+L ESP_WeatherStation-v2.0-rescue:MaxNil_components_BMP280-ESP_WeatherStation_v2.0-cache U4
 U 1 1 5A9331AD
 P 7350 1500
@@
 $EndComp
 $Comp
-L ESP_WeatherStation-rescue:ESP-12F U2
+L ESP8266:ESP-12F U2
 U 1 1 5A92C426
 P 4200 2600
